Commit message: moved all structural data to urdf file

File: description/roboraider.urdf (robot description, URDF)
Before this commit: robot RoboRaider, 1 links, 0 joints
Links:
- added link orbbec_sensor_frame
- added link rplidar_sensor_frame
- added link sonar_sensor_frame
- link base_link: mass 4.0 -> None; geometry collision box size=0.360 0.380 0.330; visual mesh filename=package://roboraider/description/RoboRaiderGeometry_body.stl
Joints:
- added joint base_to_orbbec_sensor_frame: type fixed, parent base_link, child orbbec_sensor_frame, origin xyz=-0.112 0.0375 0.3175
- added joint base_to_rplidar_sensor_frame: type fixed, parent base_link, child rplidar_sensor_frame, origin xyz=0.075 0 0.2193 rpy=0 0 3.1415927
- added joint base_to_sonar_sensor_frame: type fixed, parent base_link, child sonar_sensor_frame, origin xyz=0.16 0.0 0.065
